Commit message: パラメータの変更

File: urdf/wheel/wheel_urdf.xacro (robot description, xacro)
@@ -28,5 +28,5 @@
       <inertial>
         <origin xyz="0 0 0" rpy="-${M_PI/2} 0 0"/>
-				<mass value="0.3"/>
+				<mass value="3.0"/>
         <inertia ixx="7.0238032e-6" ixy="0.0" ixz="-8.4978788e-11" iyy="3.5665783e-6" iyz="-2.2592014e-12" izz="3.5673196e-6"/>
       </inertial>
