Commit message: Noeticに対応。PIDパラメータが設定されていない問題を修正

File: robots/lightrover_urdf.xacro (robot description, xacro)
@@ -1,4 +1,4 @@
 <?xml version="1.0"?>
-<robot name="fourth_robot" xmlns:xacro="http://ros.org/wiki/xacro">
+<robot name="lightrover" xmlns:xacro="http://ros.org/wiki/xacro">
   <xacro:include filename="$(find lightrover_description)/urdf/common.xacro"/>
   <xacro:include filename="$(find lightrover_description)/urdf/base/base_urdf.xacro"/>

File: urdf/base/base_urdf.xacro (robot description, xacro)
@@ -22,5 +22,5 @@
       <inertial>
         <origin xyz="-0.025 0.0 0.024" rpy="0.0 0.0 0.0"/>
-        <mass value="2.0"/>
+        <mass value="0.0020"/>
         <inertia ixx="8.0206480e-4" ixy="3.2953465e-5" ixz="3.1434721e-5" iyy="9.0126446e-4" iyz="-1.2433875e-4" izz="6.4944281e-4"/>
       </inertial>

File: urdf/common.xacro (robot description, xacro)
@@ -1,4 +1,4 @@
 <?xml version="1.0"?>
 <robot xmlns:xacro="http://ros.org/wiki/xacro">
-  <property name="M_PI" value="3.14159274"/>
+  <xacro:property name="M_PI" value="3.14159274"/>
 </robot>

File: urdf/lidar/lidar_urdf.xacro (robot description, xacro)
@@ -5,5 +5,5 @@
   <xacro:macro name="lidar" params="prefix parent *joint_origin">
 		<joint name="${prefix}_lidar_joint" type="fixed">
-	  	<insert_block name="joint_origin"/>
+	  	<xacro:insert_block name="joint_origin"/>
 	  	<parent link="${parent}"/>
 	  	<child link="lidar_link"/>

File: urdf/wheel/wheel_urdf.xacro (robot description, xacro)
@@ -4,11 +4,11 @@
   <xacro:include filename="$(find lightrover_description)/urdf/wheel/wheel_transmission.xacro"/>
   <xacro:include filename="$(find lightrover_description)/urdf/wheel/wheel_gazebo.xacro"/>
-  <property name="wheel_radius" value="0.03"/>
-  <property name="wheel_length" value="0.005"/>
-  <property name="wheel_mass" value="0.00135"/>
-  <xacro:macro name="wheel" params="prefix parent *joint_origin *joint_axis">
+  <xacro:property name="wheel_radius" value="0.03"/>
+  <xacro:property name="wheel_length" value="0.005"/>
+  <xacro:property name="wheel_mass" value="0.0135"/>
+  <xacro:macro name="wheel" params="prefix parent *origin *axis">
     <joint name="${prefix}_wheel_joint" type="continuous">
-      <insert_block name="joint_origin"/>
-      <insert_block name="joint_axis"/>
+      <xacro:insert_block name="origin"/>
+      <xacro:insert_block name="axis"/>
       <parent link="${parent}"/>
       <child link="${prefix}_wheel_link"/>
@@ -28,5 +28,5 @@
       <inertial>
         <origin xyz="0 0 0" rpy="-${M_PI/2} 0 0"/>
-				<mass value="3.0"/>
+				<mass value="2.0"/>
         <inertia ixx="7.0238032e-6" ixy="0.0" ixz="-8.4978788e-11" iyy="3.5665783e-6" iyz="-2.2592014e-12" izz="3.5673196e-6"/>
       </inertial>
