Commit message: ros2 humbleに対応

File: urdf/lidar/lidar_gazebo.xacro (robot description, xacro)
@@ -2,5 +2,5 @@
 <robot xmlns:xacro="http://ros.org/wiki/xacro">
   <xacro:macro name="lidar_gazebo" params="prefix min_rad max_rad min_range max_range">
-	<gazebo reference="lidar_link">
+	<gazebo reference="laser_frame">
       <sensor type="ray" name="${prefix}_lidar_sensor">
 		<pose>0 0 0 0 0 0</pose>
@@ -29,5 +29,5 @@
 		<plugin name="gazebo_ros_${prefix}_lidar_controller" filename="libgazebo_ros_laser.so">
           <topicName>/scan</topicName>
-          <frameName>lidar_link</frameName>
+          <frameName>laser_frame</frameName>
 		</plugin>
       </sensor>

File: urdf/lidar/lidar_urdf.xacro (robot description, xacro)
@@ -7,7 +7,7 @@
 	  	<xacro:insert_block name="joint_origin"/>
 	  	<parent link="${parent}"/>
-	  	<child link="lidar_link"/>
+	  	<child link="laser_frame"/>
 		</joint>
-		<link name="lidar_link"/>
+		<link name="laser_frame"/>
   </xacro:macro>
 </robot>

File: urdf/lightrover_urdf.xacro (robot description, xacro)
@@ -30,5 +30,5 @@
   <!-- Lidar -->
   <xacro:lidar prefix="center" parent="base_link">
-  	<origin xyz="-0.07 0 0.086"/>
+  	<origin xyz="-0.07 0 0.086" rpy="0 0 -1.5708"/>
   </xacro:lidar>
   <!-- ===============  Transmission =============== -->
